File: Kicad/68hc11.kicad_pcb (KiCad board)
At the start: 2 copper layers, 86 x 88.3 mm, 36 parts, among them J2 Conn_01x03, J3 Conn_01x09, J4 Conn_01x03, J5 Conn_01x05, J6 Conn_01x06, U1 68HC11A8, U2 AS6C4008, U3 74HCT573, U4 74HCT139, U5 27C256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

Commit message: Updated to KiCad 6.0
Added new 3d models among other settings
Connections:
- U4 pad 12: (no net) -> unconnected-(U4-Pad12)
- U4 pad 4: (no net) -> unconnected-(U4-Pad4)
- U4 pad 5: (no net) -> unconnected-(U4-Pad5)
- U4 pad 6: (no net) -> unconnected-(U4-Pad6)
- U7 pad 11: (no net) -> unconnected-(U7-Pad11)
- U7 pad 6: (no net) -> unconnected-(U7-Pad6)
- U7 pad 8: (no net) -> unconnected-(U7-Pad8)
Other:
- net class Default removed
- net class Power removed
