File: Kicad/68hc11.kicad_sch (KiCad schematic)
At the start: 36 parts, among them J2 Conn_01x03, J3 Conn_01x09, J4 Conn_01x03, J5 Conn_01x05, J6 Conn_01x06, U1 68HC11A8, U2 AS6C4008, U3 74HCT573, U4 74HCT139, U5 27C256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

Commit message: Updated to KiCad 6.0
Added new 3d models among other settings
Changed lines of the file:
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@@
       (effects (font (size 1.27 1.27)) (justify left))
     )
-    (property "Footprint" "Housings_DIP:DIP-32_W15.24mm" (id 2) (at 294.64 113.03 0)
-      (effects (font (size 1.27 1.27)) hide)
-    )
+    (property "Footprint" "Housings_DIP:DIP-32_W15.24mm" (id 2) (at 294.64 113.03 0))
     (property "Datasheet" "" (id 3) (at 294.64 113.03 0)
       (effects (font (size 1.27 1.27)) hide)
